File: battle bunnies.brd (EAGLE design)
At the start: 151.7 x 94 mm, 59 parts, among them IC1 CP2104, Q1 mmbt2222, Q2 mmbt2222, SW2 KMR2, U1 PCA9685, U2 SPX3819, U3 MCP73831T-2ACI/OT, X2 ESP-12, X4 20329

Commit message: Re-working for amica module
Parts:
- removed C3, C6, C8: 10µF, microbuilder:0805-NO
- removed C7: 1uF, microbuilder:0603-NO
- removed CHG: ORANGE, microbuilder:CHIPLED_0805_NOOUTLINE
- removed D2: Yellow, SparkFun-LED:LED-0603
- removed D4: RED, SparkFun-LED:LED-0603
- removed D5: GREEN, SparkFun-LED:LED-0603
- removed IC1: CP2104, microbuilder:QFN24_4MM_SMSC
- removed Q1, Q2: mmbt2222, SparkFun:SOT23-3
- removed R1, R15: 1K, SparkFun-Resistors:0603-RES
- removed R12: 1K, microbuilder:_0603MP
- removed R16: 200, SparkFun-Resistors:0603-RES
- removed R2: 1K, microbuilder:0603-NO
- removed R3, R4, R5, R9: 10K, microbuilder:0603-NO
- removed R6: 4.7K, microbuilder:0603-NO
- removed R7: 10K, microbuilder:_0603MP
- removed R8: 2.0K\, microbuilder:0603-NO
- removed S1: (no value), SparkFun-Electromechanical:SWITCH-SPST-SMD-A
- removed SJ1: (no value), microbuilder:SOLDERJUMPER_CLOSEDWIRE@1
- removed SW2: KMR2, microbuilder:BTN_KMR2_4.6X2.8
- removed U2: SPX3819, microbuilder:SOT23-5
- removed U3: MCP73831T-2ACI/OT, microbuilder:SOT23-5
- removed X2: ESP-12, microbuilder:ESP-12E
- removed X4: 20329, microbuilder:4UCONN_20329_V2
- added AMICA-NODEMCU: ESP12E_DEVKIT, ESP12E_DEVKIT:ESP12E_DEVKIT
- RN2: value 220 -> (none)
- RN3: value 10K -> (none)
- U$31: value AA1 -> AAA3NOHOLES; device Electromechanical:AA1 -> Warthog9-Batteries:AAA3-NOHOLES
- moved D1 12.5 mm to (30.1, 15.2), turned to 180 degrees
- moved U$31 7.86 mm to (26.0, 43.5)
Connections:
- removed net DTR: IC1.23, Q2.2, R5.1
- removed net N$1: CHG.C, R2.1
- removed net N$10: D2.A, R15.2
- removed net N$11: D4.A
- removed net N$12: Q1.1, R5.2
- removed net N$13: Q2.1, R7.2
- removed net N$3: R2.2, U3.1
- removed net N$4: D4.C, R16.1
- removed net N$8: D5.A, R1.2
- removed net N$9: SJ1.1, U3.3
- removed net RTS: IC1.19, Q1.2, R7.1
- removed net RXLED: D2.C, IC1.13
- removed net TXLED: D5.C, IC1.14
- removed net USBD_N: IC1.4, X4.D-
- removed net USBD_P: IC1.3, X4.D+
- removed net USB_RX: IC1.21, R12.1
- removed net VBAT: C3.1, D1.A, SJ1.2, U$31.POS
- removed net VBUS: C6.1, CHG.A, D1.C, IC1.8, S1.3, U2.1, U3.4, X4.VBUS
- new net GPIO10: AMICA-NODEMCU.SD3
- new net GPIO9: AMICA-NODEMCU.SD2
- new net VCC: AMICA-NODEMCU.VIN, D1.C
- net 3.3V: now also AMICA-NODEMCU.3V3@0, AMICA-NODEMCU.3V3@1, AMICA-NODEMCU.3V3@2; no longer C7.1, C8.1, IC1.5, IC1.6, IC1.7, R1.1, R15.1, R3.2, R4.2, R9.2, U2.5, X2.8
- net ADC: now also AMICA-NODEMCU.AD0; no longer X2.2
- net CH_PD: no longer R3.1, X2.3
- net EN: now also AMICA-NODEMCU.EN; no longer S1.2, U2.3
- net GND: now also AMICA-NODEMCU.GND@0, AMICA-NODEMCU.GND@1, AMICA-NODEMCU.GND@2, AMICA-NODEMCU.GND@3; no longer C3.2, C6.2, C7.2, C8.2, IC1.2, IC1.THERM, R16.2, R6.1, R8.2, S1.1, SW2.A, SW2.A', U2.2, U3.2, X2.9, X4.BASE@1, X4.BASE@2, X4.GND, X4.SPRT@1, X4.SPRT@2, X4.SPRT@3, X4.SPRT@4
- net GPIO0: now also AMICA-NODEMCU.D3; no longer Q2.3, X2.12
- net GPIO12/MISO: now also AMICA-NODEMCU.D6; no longer X2.6
- net GPIO13/MOSI: now also AMICA-NODEMCU.D7; no longer X2.7
- net GPIO14/SCK: now also AMICA-NODEMCU.D5; no longer X2.5
- net GPIO15: now also AMICA-NODEMCU.D8; no longer R6.2, X2.10
- net GPIO16: now also AMICA-NODEMCU.D0; no longer X2.4
- net GPIO2: now also AMICA-NODEMCU.D4; no longer R9.1, X2.11
- net GPIO4/SDA: now also AMICA-NODEMCU.D2; no longer X2.13
- net GPIO5/SCL: now also AMICA-NODEMCU.D1; no longer X2.14
- net N$2: now also D1.A, U$31.POS; no longer R8.1, U3.5
- net RESET: now also AMICA-NODEMCU.RST; no longer Q1.3, R4.1, SW2.B, SW2.B', X2.1
- net RXD: now also AMICA-NODEMCU.RX; no longer R12.2, X2.15
- net TXD: now also AMICA-NODEMCU.TX; no longer IC1.20, X2.16
Routing:
- net VBUS: track 98.2 -> 0.00 mm, vias 5 -> 0
- net CH_PD: track 109.0 -> 43.7 mm, vias 3 -> 2
- net RTS: track 52.7 -> 0.00 mm, vias 4 -> 0
- net USB_RX: track 51.0 -> 0.00 mm, vias 2 -> 0
- net DTR: track 49.3 -> 0.00 mm
- net RXD: track 122.6 -> 161.9 mm
- net USBD_N: track 37.5 -> 0.00 mm, vias 2 -> 0
- net USBD_P: track 37.3 -> 0.00 mm
- net GPIO12/MISO: track 130.9 -> 163.6 mm, vias 1 -> 3
- net ADC: track 111.9 -> 135.9 mm
- net RXLED: track 23.3 -> 0.00 mm, vias 1 -> 0
- net VBAT: track 22.8 -> 0.00 mm, vias 1 -> 0
- net N$3: track 20.4 -> 0.00 mm, vias 2 -> 0
- net GPIO15: track 93.5 -> 113.5 mm, vias 3 -> 1
- net TXLED: track 19.9 -> 0.00 mm, vias 1 -> 0
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- removed copper zone on layer 16, net GND
- removed copper zone on layer 16, net VBUS
Other:
- board size 151.7 x 94 mm -> 151.7 x 95.1 mm
- board text removed: "Chg"
- board text removed: "Reset"
- board text removed: "Rx"
- board text removed: "TX"
