File: battle bunnies.brd (EAGLE design)
At the start: 151.7 x 94 mm, 59 parts, among them IC1 CP2104, Q1 mmbt2222, Q2 mmbt2222, SW2 KMR2, U1 PCA9685, U2 SPX3819, U3 MCP73831T-2ACI/OT, X2 ESP-12, X4 20329

Commit message: USB: Swapping the USB part out - twas unobtanium
The 4UCONN connector that Adafruit used is basically made of unobtanium
and more or less doesn't exist.  The part that was trying to be used
the rear prongs did not match up by any stretch of the imagination.

A mess of e-mails an annoyance ensued.

I'm swapping out the part on everything I can now, this seems to be
more common, and there's parts that are similar enough to it that
replacing it won't be a big deal.  New part is the
Amphenol FCI 10118193-0001LF
Parts:
- X4: device microbuilder:4UCONN_20329_V2 -> microbuilder:MICRO-USB5+6P-SMD-0.65-B
- moved X4 1.19 mm to (21.3, 6.64)
Connections:
- net GND: now also X4.5, X4.S1, X4.S2, X4.S3, X4.S4, X4.S5, X4.S6; no longer X4.BASE@1, X4.BASE@2, X4.GND, X4.SPRT@1, X4.SPRT@2, X4.SPRT@3, X4.SPRT@4
- net USBD_N: now also X4.2; no longer X4.D-
- net USBD_P: now also X4.3; no longer X4.D+
- net VBUS: now also X4.1; no longer X4.VBUS
Changed lines of the file:
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@@
 <layer number="59" name="tCarbon" color="7" fill="1" visible="no" active="no"/>
 <layer number="60" name="bCarbon" color="7" fill="1" visible="no" active="no"/>
+<layer number="88" name="SimResults" color="7" fill="1" visible="yes" active="yes"/>
+<layer number="89" name="SimProbes" color="7" fill="1" visible="yes" active="yes"/>
 <layer number="90" name="Modules" color="5" fill="1" visible="no" active="no"/>
 <layer number="91" name="Nets" color="2" fill="1" visible="no" active="no"/>
@@
 <layer number="115" name="ReferenceISLANDS" color="7" fill="1" visible="yes" active="yes"/>
 <layer number="116" name="Patch_BOT" color="9" fill="4" visible="yes" active="yes"/>
+<layer number="117" name="BACKMAAT1" color="7" fill="1" visible="no" active="no"/>
 <layer number="118" name="Rect_Pads" color="7" fill="1" visible="yes" active="yes"/>
+<layer number="119" name="KAP_TEKEN" color="7" fill="1" visible="no" active="no"/>
+<layer number="120" name="KAP_MAAT1" color="7" fill="1" visible="no" active="no"/>
 <layer number="121" name="_tsilk" color="7" fill="1" visible="yes" active="yes"/>
 <layer number="122" name="_bsilk" color="7" fill="1" visible="yes" active="yes"/>
@@
 <layer number="128" name="_bValues" color="7" fill="1" visible="yes" active="yes"/>
 <layer number="129" name="Mask" color="7" fill="1" visible="yes" active="yes"/>
+<layer number="130" name="SMDSTROOK" color="7" fill="1" visible="no" active="no"/>
 <layer number="131" name="tAdjust" color="7" fill="1" visible="yes" active="yes"/>
 <layer number="132" name="bAdjust" color="7" fill="1" visible="yes" active="yes"/>
+<layer number="133" name="bottom_silk" color="7" fill="1" visible="no" active="no"/>
 <layer number="144" name="Drill_legend" color="7" fill="1" visible="yes" active="yes"/>
+<layer number="145" name="DrillLegend_01-16" color="7" fill="1" visible="yes" active="yes"/>
 <layer number="150" name="Notes" color="7" fill="1" visible="yes" active="yes"/>
 <layer number="151" name="HeatSink" color="7" fill="1" visible="yes" active="yes"/>
@@
 <element name="U3" library="microbuilder" package="SOT23-5" value="MCP73831T-2ACI/OT" x="31.496" y="26.67" rot="MR0"/>
 <element name="X2" library="microbuilder" package="ESP-12E" value="ESP-12" x="41.5925" y="63.1825"/>
-<element name="X4" library="microbuilder" package="4UCONN_20329_V2" value="20329" x="21.2725" y="5.4483" rot="MR0"/>
+<element name="X4" library="microbuilder" package="MICRO-USB5+6P-SMD-0.65-B" value="20329" x="21.2725" y="6.638925" rot="MR0"/>
 <element name="JP2" library="pinhead" package="1X15" value="" x="129.54" y="41.91" rot="R180"/>
 <element name="JP4" library="pinhead" package="1X15" value="" x="127.9525" y="87.3125" smashed="yes" rot="R180">
@@
 <contactref element="SW2" pad="A"/>
 <contactref element="SW2" pad="A'"/>
-<contactref element="X4" pad="BASE@1"/>
-<contactref element="X4" pad="BASE@2"/>
-<contactref element="X4" pad="GND"/>
-<contactref element="X4" pad="SPRT@1"/>
-<contactref element="X4" pad="SPRT@2"/>
-<contactref element="X4" pad="SPRT@3"/>
-<contactref element="X4" pad="SPRT@4"/>
+<contactref element="X4" pad="5"/>
 <contactref element="IC1" pad="2"/>
 <contactref element="IC1" pad="THERM"/>
@@
 <wire x1="8.796378125" y1="21.564078125" x2="7.73571875" y2="21.564078125" width="0.1524" layer="16"/>
 <wire x1="56.911875" y1="55.483125" x2="55.641875" y2="55.50625" width="0.1524" layer="16"/>
+<contactref element="X4" pad="S1"/>
+<contactref element="X4" pad="S2"/>
+<contactref element="X4" pad="S3"/>
+<contactref element="X4" pad="S4"/>
+<contactref element="X4" pad="S5"/>
+<contactref element="X4" pad="S6"/>
 </signal>
 <signal name="N$4">
@@
 <contactref element="U3" pad="4"/>
 <contactref element="CHG" pad="A"/>
-<contactref element="X4" pad="VBUS"/>
+<contactref element="X4" pad="1"/>
 <contactref element="IC1" pad="8"/>
 <wire x1="29.21" y1="15.71625" x2="29.21" y2="26.6341" width="0.4064" layer="16"/>
@@
 <vertex x="27.94" y="27.94"/>
 </polygon>
-<wire x1="22.5725" y1="6.2233" x2="22.5425" y2="7.77875" width="0.4064" layer="16"/>
 <via x="22.5425" y="7.77875" extent="1-16" drill="0.3048" diameter="0.3048"/>
 <wire x1="22.5425" y1="7.77875" x2="26.67225" y2="7.77875" width="0.4064" layer="1"/>
@@
 <wire x1="7.3025" y1="18.0975" x2="7.62" y2="18.0975" width="0.3048" layer="16"/>
 <wire x1="6.35" y1="19.05" x2="6.8518375" y2="19.5518375" width="0" layer="19" extent="16-16"/>
+<wire x1="22.5725" y1="6.388925" x2="22.5725" y2="7.74875" width="0.3048" layer="16"/>
+<wire x1="22.5725" y1="7.74875" x2="22.5425" y2="7.77875" width="0.3048" layer="16"/>
 </signal>
 <signal name="VBAT">
@@
 </signal>
 <signal name="USBD_P" class="1">
-<contactref element="X4" pad="D+"/>
+<contactref element="X4" pad="3"/>
 <contactref element="IC1" pad="3"/>
-<wire x1="21.4376" y1="6.19125" x2="21.30455" y2="6.19125" width="0.1524" layer="16"/>
-<wire x1="21.30455" y1="6.19125" x2="21.2725" y2="6.2233" width="0.1524" layer="16"/>
 <via x="21.59" y="9.8425" extent="1-16" drill="0.3048"/>
-<wire x1="21.4376" y1="6.19125" x2="21.4376" y2="8.0899" width="0.1524" layer="16"/>
 <via x="20.32" y="9.8425" extent="1-16" drill="0.3048"/>
 <wire x1="20.32" y1="9.8425" x2="21.59" y2="9.8425" width="0.1524" layer="1"/>
@@
 <wire x1="9.8425" y1="19.58303125" x2="9.8425" y2="19.81085" width="0.1524" layer="16"/>
 <wire x1="9.8425" y1="19.81085" x2="9.326709375" y2="20.326640625" width="0.1524" layer="16"/>
-<wire x1="21.4376" y1="8.0899" x2="20.955" y2="8.5725" width="0.1524" layer="16"/>
-<wire x1="20.955" y1="8.5725" x2="20.955" y2="9.2075" width="0.1524" layer="16"/>
+<wire x1="20.955" y1="8.2423" x2="20.955" y2="9.2075" width="0.1524" layer="16"/>
 <wire x1="20.955" y1="9.2075" x2="21.59" y2="9.8425" width="0.1524" layer="16"/>
 <wire x1="19.58303125" y1="9.8425" x2="20.32" y2="9.8425" width="0.1524" layer="16"/>
+<wire x1="21.2725" y1="7.9248" x2="21.2725" y2="6.388925" width="0.1524" layer="16"/>
+<wire x1="21.2725" y1="7.9248" x2="20.955" y2="8.2423" width="0.1524" layer="16"/>
 </signal>
 <signal name="USBD_N" class="1">
-<contactref element="X4" pad="D-"/>
+<contactref element="X4" pad="2"/>
 <contactref element="IC1" pad="4"/>
 <via x="21.59" y="8.89" extent="1-16" drill="0.3048"/>
-<wire x1="21.9225" y1="6.2233" x2="21.7424" y2="6.5558" width="0.1524" layer="16"/>
 <via x="20.32" y="8.89" extent="1-16" drill="0.3048"/>
 <wire x1="20.10446875" y1="8.89" x2="10.052234375" y2="18.942234375" width="0.1524" layer="16"/>
 <wire x1="10.052234375" y1="18.942234375" x2="8.97315625" y2="19.9730875" width="0.1524" layer="16"/>
 <wire x1="20.10446875" y1="8.89" x2="20.32" y2="8.89" width="0.1524" layer="16"/>
-<wire x1="21.7424" y1="6.5558" x2="21.7424" y2="8.0899" width="0.1524" layer="16"/>
 <wire x1="21.59" y1="8.89" x2="22.06625" y2="8.89" width="0.1524" layer="16"/>
 <wire x1="22.06625" y1="8.89" x2="22.225" y2="8.73125" width="0.1524" layer="16" curve="-90"/>
 <wire x1="22.225" y1="8.73125" x2="22.225" y2="8.5725" width="0.1524" layer="16"/>
-<wire x1="22.225" y1="8.5725" x2="21.7424" y2="8.0899" width="0.1524" layer="16"/>
 <wire x1="20.32" y1="8.89" x2="21.59" y2="8.89" width="0.1524" layer="1"/>
+<wire x1="21.9225" y1="8.27" x2="21.9225" y2="6.388925" width="0.1524" layer="16"/>
+<wire x1="21.9225" y1="8.27" x2="22.225" y2="8.5725" width="0.1524" layer="16"/>
 </signal>
 <signal name="RTS">
