File: battle bunnies.sch (EAGLE design)
At the start: 59 parts, among them IC1 CP2104, Q1 mmbt2222, Q2 mmbt2222, SW2 KMR2, U1 PCA9685, U2 SPX3819, U3 MCP73831T-2ACI/OT, X2 ESP-12, X4 20329

Commit message: Re-working for amica module
Parts:
- removed C3, C6, C8: 10µF, microbuilder:CAP_CERAMIC0805-NOOUTLINE
- removed C7: 1uF, microbuilder:CAP_CERAMIC0603_NO
- removed CHG: ORANGE, microbuilder:LED0805_NOOUTLINE
- removed D2: Yellow, SparkFun-LED:LED-YELLOW0603
- removed D4: RED, SparkFun-LED:LED-RED0603
- removed D5: GREEN, SparkFun-LED:LED-GREEN0603
- removed IC1: CP2104, microbuilder:CP2104
- removed Q1, Q2: mmbt2222, SparkFun:TRANSISTOR_NPNSOT23-3
- removed R1, R15: 1K, SparkFun-Resistors:1KOHM-1/10W-1%(0603)
- removed R12: 1K, microbuilder:RESISTOR_0603MP
- removed R16: 200, SparkFun-Resistors:200OHM1/10W1%(0603)
- removed R2: 1K, microbuilder:RESISTOR_0603_NOOUT
- removed R3, R4, R5, R9: 10K, microbuilder:RESISTOR_0603_NOOUT
- removed R6: 4.7K, microbuilder:RESISTOR_0603_NOOUT
- removed R7: 10K, microbuilder:RESISTOR_0603MP
- removed R8: 2.0K\, microbuilder:RESISTOR_0603_NOOUT
- removed S1: (no value), SparkFun-Electromechanical:SWITCH-SPDT-SMD-A
- removed SJ1: (no value), microbuilder:SOLDERJUMPER_CLOSED
- removed SW2: KMR2, microbuilder:SWITCH_TACT_SMT4.6X2.8
- removed U2: SPX3819, microbuilder:VREG_SOT23-5
- removed U3: MCP73831T-2ACI/OT, microbuilder:MCP73831/2
- removed X2: ESP-12, microbuilder:ESP-12E
- removed X4: 20329, microbuilder:USB_MICRO_20329_V2
- added AMICA-NODEMCU: ESP12E_DEVKIT, ESP12E_DEVKIT:ESP12E_DEVKIT
- RN2: value 220 -> (none)
- RN3: value 10K -> (none)
- U$31: value AA1 -> AAA3NOHOLES; device Electromechanical:AA1 -> Warthog9-Batteries:AAA3NOHOLES
Connections:
- removed net DTR: IC1G$1.DTR, Q2.E, R5.1
- removed net N$1: CHG.C, R2.1
- removed net N$10: D2.A, R15.2
- removed net N$11: D4.A
- removed net N$12: Q1.B, R5.2
- removed net N$13: Q2.B, R7.2
- removed net N$3: R2.2, U3.STAT
- removed net N$4: D4.C, R16.1
- removed net N$8: D5.A, R1.2
- removed net N$9: SJ1.1, U3.VBAT
- removed net RTS: IC1G$1.RTS, Q1.E, R7.1
- removed net RXLED: D2.C, IC1G$1.GPIO1/RXLED
- removed net TXLED: D5.C, IC1G$1.GPIO0/TXLED
- removed net USBD_N: IC1G$1.D-, X4.D-
- removed net USBD_P: IC1G$1.D+, X4.D+
- removed net USB_RX: IC1G$1.TXD, R12.1
- removed net VBAT: C3.1, D1.A, SJ1.2, U$31.+
- removed net VBUS: C6.1, CHG.A, D1.C, IC1G$1.VBUS, S1.S, U2.IN, U3.VDD, X4.VBUS
- new net GPIO10: AMICA-NODEMCU.SD3
- new net GPIO9: AMICA-NODEMCU.SD2
- new net VCC: AMICA-NODEMCU.VIN, D1.C
- net 3.3V: now also AMICA-NODEMCU.3V3@0, AMICA-NODEMCU.3V3@1, AMICA-NODEMCU.3V3@2; no longer C7.1, C8.1, IC1G$1.REGIN, IC1G$1.VDD, IC1G$1.VIO, R1.1, R15.1, R3.2, R4.2, R9.2, U2.OUT, X2.VCC
- net ADC: now also AMICA-NODEMCU.AD0; no longer X2.ADC
- net CH_PD: no longer R3.1, X2.CH_PD
- net EN: now also AMICA-NODEMCU.EN; no longer S1.P, U2.EN
- net GND: now also AMICA-NODEMCU.GND@0, AMICA-NODEMCU.GND@1, AMICA-NODEMCU.GND@2, AMICA-NODEMCU.GND@3; no longer C3.2, C6.2, C7.2, C8.2, IC1G$1.GND, IC1G$2.TP, R16.2, R6.1, R8.2, S1.O, SW2.P, SW2.P1, U2.GND, U3.VSS, X2.GND, X4.GND
- net GPIO0: now also AMICA-NODEMCU.D3; no longer Q2.C, X2.GPIO0
- net GPIO12/MISO: now also AMICA-NODEMCU.D6; no longer X2.GPIO12
- net GPIO13/MOSI: now also AMICA-NODEMCU.D7; no longer X2.GPIO13
- net GPIO14/SCK: now also AMICA-NODEMCU.D5; no longer X2.GPIO14
- net GPIO15: now also AMICA-NODEMCU.D8; no longer R6.2, X2.GPIO15
- net GPIO16: now also AMICA-NODEMCU.D0; no longer X2.GPIO16
- net GPIO2: now also AMICA-NODEMCU.D4; no longer R9.1, X2.GPIO2
- net GPIO4/SDA: now also AMICA-NODEMCU.D2; no longer X2.GPIO4
- net GPIO5/SCL: now also AMICA-NODEMCU.D1; no longer X2.GPIO5
- net N$2: now also D1.A, U$31.+; no longer R8.1, U3.PROG
- net RESET: now also AMICA-NODEMCU.RST; no longer Q1.C, R4.1, SW2.S, SW2.S1, X2.RESET
- net RXD: now also AMICA-NODEMCU.RX; no longer R12.2, X2.RXD
- net TXD: now also AMICA-NODEMCU.TX; no longer IC1G$1.RXD, X2.TXD
Other:
- note added: "Use AAA 1.5V Batteries"
- note removed: "1.0K = 1000mA"
- note removed: "10K = 100mA"
- note removed: "2.0K = 500mA"
- note removed: "5.0K = 200mA"
- note removed: "LIPO CHARGING"
- note removed: "Power "On" Indicator"
- note removed: "RESET"
- note removed: "USB TO SERIAL CONVERTER"
- note removed: "Use 14500 3.7V Batteries"
- moved on the sheet: D1
